File: hw/_module_core.sch (KiCad schematic (older format))
At the start: 41 parts, among them J10 Conn_Left, J11 Conn_Right, J2 power_bus, SW1 reset, U1 ProMicro, U2 LM78L05_TO92, U3 TL074, U4 TL074

Commit message: worked on the PCB. - adjusted CV scale parameters - removed debug code
Connections:
- net cv_select_in: now also U1.20 (21); no longer U1.7 (4)
Other:
- note removed: "random seed"
Changed lines of the file:
@@
 	7450 3050 7000 3050
 NoConn ~ 5450 4650
-NoConn ~ 6650 3750
 Text Label 6650 4200 0    50   ~ 0
 cv_len
@@
 Text Label 6650 3900 0    50   ~ 0
 cv_sft
-Text Label 5450 4050 2    50   ~ 0
+Text Label 6650 3750 0    50   ~ 0
 cv_select_in
-Text Notes 7200 3750 2    50   ~ 0
-random seed
 Wire Wire Line
 	7450 3450 6650 3450
@@
 	1750 1100 1750 1500
 Connection ~ 1750 1100
+NoConn ~ 5450 4050
 $EndSCHEMATC
